Commit message: fixed gazebo sensors and added new gazebo world

File: evarobot_description/urdf/evarobot.urdf (robot description, URDF)
Before this commit: robot evarobot, 17 links, 16 joints
Links:
- added link kinect_dummy
- link base_link: geometry collision box size=0.25 0.251 0.3005; visual mesh filename=package://evarobot_description/meshes/evarobot_all.stl scale=0.001 0.001 0.001
Joints:
- added joint kinect_joint_dummy: type fixed, parent evarobot/kinect_link, child kinect_dummy, origin xyz=0 0 0 rpy=-1.57 0 -1.57, axis 0 1 0
