Commit message: delete unused lines

File: evarobot_description/urdf/evarobot_lidar.urdf.xacro (robot description, xacro)
@@ -63,5 +63,4 @@
 				</ray>
     			<plugin name="${prefix}_controller" filename="libgazebo_ros_gpu_laser.so">
-<!--					<robotNamespace>${robot_namespace}</robotNamespace> -->
 					<topicName>${topic_name}</topicName>
 					<frameName>${frame_name}</frameName>
@@ -69,11 +68,4 @@
 			</sensor>
 		</gazebo>
-<!--
-		<gazebo>
-			<plugin name="${prefix}_control" filename="libgazebo_ros_control.so">
-				<robotNamespace>${robot_namespace}</robotNamespace>
-			</plugin>
-		</gazebo>
--->
 	</xacro:macro>
 </robot>

File: evarobot_description/urdf/evarobot_wheel.urdf.xacro (robot description, xacro)
@@ -13,5 +13,5 @@
 				<geometry>
 					<cylinder length="${cylinder_length}" radius="${cylinder_radius}"/>
-					<mesh filename="model://evarobot/meshes/wheel.stl" scale="0.001 0.001 0.001"/>
+					<mesh filename="model://evarobot/meshes/wheel.dae" scale="0.001 0.001 0.001"/>
 				</geometry>
 				<material name="black"/>
