Commit message: ...

File: evarobot_description/urdf/evarobot.urdf.xacro (robot description, xacro)
@@ -84,5 +84,5 @@
 						 parent_link="base_link" />
   <!-- Lidar -->
-  <xacro:evarobot_lidar prefix="sensor/lidar"
+<!--  <xacro:evarobot_lidar prefix="sensor/lidar"
                         joint_x="-0.09"
                         joint_y="0.0"
@@ -103,4 +103,5 @@
 												topic_name="lidar"
 												frame_name="sensor/lidar_link" />
+												-->
 <!--
   <xacro:evarobot_lidar prefix="sensor/lidar"
@@ -124,12 +125,13 @@
 												frame_name="sensor/lidar_link" />
 -->
+				<!-- joint_z="0.112" -->
   <!-- Kinect -->
    <xacro:evarobot_kinect prefix="sensor/kinect"
 						 joint_x="0.0"
 						 joint_y="0.0"
-						 joint_z="0.112"
-						 joint_roll="0.0"
+						 joint_z="0.23"
+						 joint_roll="-1.57"
 						 joint_pitch="0.0"
-						 joint_yaw="0.0"
+						 joint_yaw="-1.57"
 						 parent_link="base_link"
 						 base_line="0.2"

File: evarobot_description/urdf/evarobot_kinect.urdf.xacro (robot description, xacro)
@@ -9,5 +9,5 @@
 			">
 		<!-- Kinect Link -->
-		<link name="${prefix}_link">
+		<link name="kinect_dummy">
 			<collision>
 				<origin xyz="0 0 0" rpy="0 0 0"/>
@@ -33,8 +33,8 @@
 			<origin xyz="${joint_x} ${joint_y} ${joint_z}" rpy="0 0 0"/>
 			<parent link="${parent_link}"/>
-			<child link="${prefix}_link"/>
+			<child link="kinect_dummy"/>
 		</joint>
 		<!-- Kinect Dummy Link -->
-		<link name="kinect_dummy">
+		<link name="${prefix}_link">
 			<pose>0 0 0 0 0 0</pose>
 		</link>
@@ -42,6 +42,6 @@
 		<joint name="kinect_joint_dummy" type="fixed">
 			<origin xyz="0 0 0" rpy="${joint_roll} ${joint_pitch} ${joint_yaw}"/>
-			<parent link="${prefix}_link"/>
-			<child link="kinect_dummy"/>
+			<parent link="kinect_dummy"/>
+			<child link="${prefix}_link"/>
 			<axis xyz="0 1 0"/>
 		</joint>

Commit message: ...

File: evarobot_description/urdf/evarobot.urdf.xacro (robot description, xacro)
@@ -4,4 +4,5 @@
  -->
 <robot name="evarobot" xmlns:xacro="http://ros.org/wiki/xacro">
+  <xacro:property name="pi" value="3.1415926535897931" />
   <!-- Includes -->
   <xacro:include filename="$(find evarobot_description)/urdf/evarobot_base.urdf.xacro"/>
@@ -14,4 +15,5 @@
   <xacro:include filename="$(find evarobot_description)/urdf/evarobot_lidar.urdf.xacro"/>
   <xacro:include filename="$(find evarobot_description)/urdf/evarobot_bumper.urdf.xacro"/>
+  <xacro:include filename="$(find evarobot_description)/urdf/plates.urdf.xacro"/>
  <!-- Differential Drive Plugin -->
  <gazebo>
@@ -26,6 +28,6 @@
 	  <leftJoint>right_wheel_joint</leftJoint>
 	  <rightJoint>left_wheel_joint</rightJoint>
-	  <wheelSeparation>0.3</wheelSeparation>
-	  <wheelDiameter>0.13</wheelDiameter>
+	  <wheelSeparation>0.33</wheelSeparation>
+	  <wheelDiameter>0.17</wheelDiameter>
 	  <wheelTorque>20</wheelTorque>
 	  <commandTopic>cmd_vel</commandTopic>
@@ -39,41 +41,53 @@
   <!-- Base -->
   <xacro:evarobot_base prefix="base"
-					   mesh_x="0.05"
-					   mesh_y="0.0"
-					   mesh_z="-0.1475"
+					   mesh_x="0.065"
+					   mesh_y="-0.11"
+					   mesh_z="-0.20"
 					   mesh_roll="0.0"
 					   mesh_pitch="0.0"
-					   mesh_yaw="1.5708"
-					   box_x="0.25"
-					   box_y="0.251"
-					   box_z="0.3005" />
+					   mesh_yaw="0"
+					   box_x="0.426"
+					   box_y="0.335"
+					   box_z="0.30" />
   <!-- Left Wheel -->
   <xacro:evarobot_wheel prefix="left_wheel"
-						joint_x="0.04975"
-						joint_y="0.1375"
-						joint_z="-0.11775"
+						joint_x="0.0"
+						joint_y="0.16"
+						joint_z="-0.1685"
 						joint_roll="0.0"
 						joint_pitch="0.0"
 						joint_yaw="0.0"
-						cylinder_length="0.024"
-						cylinder_radius="0.0675"
+						cylinder_length="0.035"
+						cylinder_radius="0.085"
 						parent_link="base_link" />
-  <!-- Right Wheel -->
+  <!-- Right Wheel 	 -->
   <xacro:evarobot_wheel prefix="right_wheel"
-						joint_x="0.04975"
-						joint_y="-0.1375"
-						joint_z="-0.11775"
+						joint_x="0.0"
+						joint_y="-0.16"
+						joint_z="-0.1685"
 						joint_roll="0.0"
 						joint_pitch="0.0"
 						joint_yaw="0.0"
-						cylinder_length="0.024"
-						cylinder_radius="0.0675"
+						cylinder_length="0.035"
+						cylinder_radius="0.085"
 						parent_link="base_link" />
   <!-- Caster -->
-  <xacro:evarobot_caster prefix="caster"
-						 radius="0.035"
-						 x="-0.1"
+  <xacro:evarobot_caster prefix="front_caster"
+						 radius="0.025"
+						 x="0.153"
 						 y="0.0"
-						 z="-0.15025"
+						 z="-0.225"
+						 roll="-1.57075"
+						 pitch="0.0"
+						 yaw="0.0"
+						 axis_x="0.577350269"
+						 axis_y="0.577350269"
+						 axis_z="0.577350269"
+						 parent_link="base_link" />
+    <xacro:evarobot_caster prefix="rear_caster"
+						 radius="0.025"
+						 x="-0.153"
+						 y="0.0"
+						 z="-0.225"
 						 roll="-1.57075"
 						 pitch="0.0"
@@ -84,8 +98,8 @@
 						 parent_link="base_link" />
   <!-- Lidar -->
-<!--  <xacro:evarobot_lidar prefix="sensor/lidar"
-                        joint_x="-0.09"
+  <xacro:evarobot_lidar prefix="sensor/lidar"
+                        joint_x="-0.15"
                         joint_y="0.0"
-                        joint_z="0.4275"
+                        joint_z="0.4415"
                         joint_roll="0.0"
                         joint_pitch="0.0"
@@ -100,35 +114,12 @@
 												range_resolution="0.1"
 												parent_link="base_link"
-												robot_namespace="evarobot"
+												robot_namespace="sensor"
 												topic_name="lidar"
-												frame_name="sensor/lidar_link" />
-												-->
-<!--
-  <xacro:evarobot_lidar prefix="sensor/lidar"
-                        joint_x="0.0"
-                        joint_y="0.0"
-                        joint_z="0.112"
-                        joint_roll="0.0"
-                        joint_pitch="0.0"
-                        joint_yaw="0.0"
-												update_rate="40"
-												samples="720"
-												resolution="1"
-												min_angle="-3.1416"
-												max_angle="3.1416"
-												min_range="0.5"
-												max_range="5.0"
-												range_resolution="0.1"
-												parent_link="base_link"
-												robot_namespace="evarobot"
-												topic_name="lidar"
-												frame_name="sensor/lidar_link" />
--->
-				<!-- joint_z="0.112" -->
+												frame_name="lidar_link" />
   <!-- Kinect -->
    <xacro:evarobot_kinect prefix="sensor/kinect"
-						 joint_x="0.0"
+						 joint_x="0.17"
 						 joint_y="0.0"
-						 joint_z="0.23"
+						 joint_z="0.16"
 						 joint_roll="-1.57"
 						 joint_pitch="0.0"
@@ -140,10 +131,4 @@
   <!-- Bumper -->
   <xacro:evarobot_bumper prefix="bumper0"
-						 joint_x="0.1575"
-						 joint_y="-0.105"
-						 joint_z="-0.1345"
-						 joint_roll="0.0"
-						 joint_pitch="0.0"
-						 joint_yaw="-0.34"
 						 box_x="0.015"
 						 box_y="0.015"
@@ -152,12 +137,8 @@
 						 parent_link="base_link"
 						 topic_name="bumper0"
-						 frame_name="bumper0_link" />
+						 frame_name="bumper0_link" >
+  <origin xyz="0.191 -0.084 -0.122" rpy="0 0 ${-pi/6}" />
+						 </xacro:evarobot_bumper>
   <xacro:evarobot_bumper prefix="bumper1"
-						 joint_x="0.1775"
-						 joint_y="0.0"
-						 joint_z="-0.1345"
-						 joint_roll="0.0"
-						 joint_pitch="0.0"
-						 joint_yaw="0.0"
 						 box_x="0.015"
 						 box_y="0.015"
@@ -166,12 +147,9 @@
 						 parent_link="base_link"
 						 topic_name="bumper1"
-						 frame_name="bumper1_link" />
+						 frame_name="bumper1_link" >
+						   <origin xyz="0.213 0.0 -0.122" rpy="0 0 0" />
+  <origin xyz="0.213 0.0 -0.122" rpy="0 0 0" />
+						</xacro:evarobot_bumper>
   <xacro:evarobot_bumper prefix="bumper2"
-						 joint_x="0.1605"
-						 joint_y="0.105"
-						 joint_z="-0.1345"
-						 joint_roll="0.0"
-						 joint_pitch="0.0"
-						 joint_yaw="0.34"
 						 box_x="0.015"
 						 box_y="0.015"
@@ -180,6 +158,8 @@
 						 parent_link="base_link"
 						 topic_name="bumper2"
-						 frame_name="bumper2_link" />
-  <!-- AHRS/IMU -->
+						 frame_name="bumper2_link" >
+  <origin xyz="0.191 0.084 -0.122" rpy="0 0 ${pi/6}" />
+						 </xacro:evarobot_bumper>
+  <!-- AHRS/IMU
   <xacro:evarobot_ahrs prefix="sensor/imu"
 					   joint_x="0.0"
@@ -195,12 +175,7 @@
 					   service_name="imu_service"
 					   robot_namespace="evarobot" />
+	-->
   <!-- Sonar -->
   <xacro:evarobot_sonar prefix="sensor/sonar0"
-						joint_x="0.14"
-						joint_y="0.0"
-						joint_z="0.0275"
-						joint_roll="0.0"
-						joint_pitch="0.0"
-						joint_yaw="0.0"
 						parent_link="base_link"
 						scan_samples="320"
@@ -213,12 +188,8 @@
 						topic_name="sonar0"
 						frame_name="sensor/sonar0_link"
-						update_rate="4" />
+						update_rate="4">
+						  <origin xyz="0.045 -0.168 0.03" rpy="0 0 ${-pi/2}" />
+  </xacro:evarobot_sonar>
   <xacro:evarobot_sonar prefix="sensor/sonar1"
-						joint_x="0.0"
-						joint_y="0.145"
-						joint_z="0.0275"
-						joint_roll="0.0"
-						joint_pitch="0.0"
-						joint_yaw="1.5708"
 						parent_link="base_link"
 						scan_samples="320"
@@ -231,12 +202,8 @@
 						topic_name="sonar1"
 						frame_name="sensor/sonar1_link"
-						update_rate="4" />
+						update_rate="4">
+								<origin xyz="0.213 0.0 0.03" rpy="0 0 0" />
+	</xacro:evarobot_sonar>
   <xacro:evarobot_sonar prefix="sensor/sonar2"
-						joint_x="-0.14"
-						joint_y="0.0"
-						joint_z="0.0275"
-						joint_roll="0.0"
-						joint_pitch="0.0"
-						joint_yaw="3.1416"
 						parent_link="base_link"
 						scan_samples="320"
@@ -249,12 +216,8 @@
 						topic_name="sonar2"
 						frame_name="sensor/sonar2_link"
-						update_rate="4" />
+						update_rate="4">
+						  <origin xyz="0.045 0.168 0.03" rpy="0 0 ${pi/2}" />
+	</xacro:evarobot_sonar>
   <xacro:evarobot_sonar prefix="sensor/sonar3"
-						joint_x="0.0"
-						joint_y="-0.145"
-						joint_z="0.0275"
-						joint_roll="0.0"
-						joint_pitch="0.0"
-						joint_yaw="-1.5708"
 						parent_link="base_link"
 						scan_samples="320"
@@ -267,13 +230,23 @@
 						topic_name="sonar3"
 						frame_name="sensor/sonar3_link"
-						update_rate="4" />
+						update_rate="4" >
+						  <origin xyz="-0.191 0.084 0.03" rpy="0 0 ${5*pi/6}" />
+	</xacro:evarobot_sonar>
+	  <xacro:evarobot_sonar prefix="sensor/sonar4"
+						parent_link="base_link"
+						scan_samples="320"
+						scan_resolution="1"
+						min_angle="-0.479965544"
+						max_angle="0.479965544"
+						range_resolution="0.01"
+						min_range="0.02"
+						max_range="5.0"
+						topic_name="sonar4"
+						frame_name="sensor/sonar4_link"
+						update_rate="4" >
+  <origin xyz="-0.191 -0.084 0.03" rpy="0 0 ${-5*pi/6}" />
+	</xacro:evarobot_sonar>
   <!-- Infrared -->
   <xacro:evarobot_infrared prefix="sensor/ir0"
-						   joint_x="0.1175"
-						   joint_y="-0.085"
-						   joint_z="-0.1075"
-						   joint_roll="0.0"
-						   joint_pitch="0.0"
-						   joint_yaw="-0.60"
 						   parent_link="base_link"
 						   scan_samples="320"
@@ -286,12 +259,8 @@
 						   topic_name="ir0"
 						   frame_name="sensor/ir0_link"
-						   update_rate="4" />
+						   update_rate="4" >
+						   	     <origin xyz="0.191 -0.084 0.03" rpy="0 0 ${-pi/6}" />
+	</xacro:evarobot_infrared>
   <xacro:evarobot_infrared prefix="sensor/ir1"
-						   joint_x="0.1475"
-						   joint_y="0.0"
-						   joint_z="-0.1075"
-						   joint_roll="0.0"
-						   joint_pitch="0.0"
-						   joint_yaw="0.0"
 						   parent_link="base_link"
 						   scan_samples="320"
@@ -304,12 +273,8 @@
 						   topic_name="ir1"
 						   frame_name="sensor/ir1_link"
-						   update_rate="4" />
+						   update_rate="4">
+						   		<origin xyz="0.191 0.084 0.03" rpy="0 0 ${pi/6}" />
+	</xacro:evarobot_infrared>
   <xacro:evarobot_infrared prefix="sensor/ir2"
-						   joint_x="0.1225"
-						   joint_y="0.085"
-						   joint_z="-0.1075"
-						   joint_roll="0.0"
-						   joint_pitch="0.0"
-						   joint_yaw="0.60"
 						   parent_link="base_link"
 						   scan_samples="320"
@@ -322,4 +287,20 @@
 						   topic_name="ir2"
 						   frame_name="sensor/ir2_link"
-						   update_rate="4" />
+						   update_rate="4">
+						   		<origin xyz="-0.045 0.168 0.03" rpy="0 0 ${pi/2}" />
+	</xacro:evarobot_infrared>
+  <xacro:evarobot_infrared prefix="sensor/ir3"
+						   parent_link="base_link"
+						   scan_samples="320"
+						   scan_resolution="1"
+						   min_angle="-0.001"
+						   max_angle="0.001"
+						   range_resolution="0.01"
+						   min_range="0.10"
+						   max_range="0.80"
+						   topic_name="ir3"
+						   frame_name="sensor/ir3_link"
+						   update_rate="4">
+						   	    <origin xyz="-0.045 -0.168 0.03" rpy="0 0 ${-pi/2}" />
+	</xacro:evarobot_infrared>
 </robot>

File: evarobot_description/urdf/evarobot_base.urdf.xacro (robot description, xacro)
@@ -4,7 +4,8 @@
 		<link name="${prefix}_link">
 			<collision>
-				<origin rpy="0 0 0" xyz="0 0 0"/>
+				<origin xyz="${mesh_x} ${mesh_y} ${mesh_z}" rpy="${mesh_roll} ${mesh_pitch} ${mesh_yaw}" />
 				<geometry>
-					<box size="${box_x} ${box_y} ${box_z}"/>
+					<mesh filename="package://evarobot_description/meshes/eva50.stl" scale="0.01 0.01 0.01"/>
+<!--				<box size="${box_x} ${box_y} ${box_z}"/> -->
 				</geometry>
 			</collision>
@@ -12,20 +13,19 @@
 				<origin xyz="${mesh_x} ${mesh_y} ${mesh_z}" rpy="${mesh_roll} ${mesh_pitch} ${mesh_yaw}" />
 				<geometry>
-					<mesh filename="package://evarobot_description/meshes/evarobot_all.stl" scale="0.001 0.001 0.001"/>
+				<!-- <box size="${box_x} ${box_y} ${box_z}"/> -->
+					<mesh filename="package://evarobot_description/meshes/eva50.stl" scale="0.01 0.01 0.01"/>
 				</geometry>
-				<material name="blue">
-					<color rgba="0 0 .8 1"/>
+				<material name="red">
+					<color rgba="0.4 0.7 .8 1"/>
 				</material>
 			</visual>
-<!--
 			<inertial>
 				<origin xyz="0 0 0" rpy="0 0 0"/>
-				<mass value="5"/>
+				<mass value="15"/>
 				<inertia
-					ixx="5.0" ixy="0.0" ixz="0.0"
-					iyy="5.0" iyz="0.0"
-					izz="5.0"/>
+					ixx="0.875" ixy="0.155" ixz="0.143"
+					iyy="0.155" iyz="0.143"
+					izz="0.143"/>
 			</inertial>
-		-->
 		</link>
 	</xacro:macro>

File: evarobot_description/urdf/evarobot_bumper.urdf.xacro (robot description, xacro)
@@ -3,5 +3,4 @@
 	<xacro:macro name="evarobot_bumper"
 	params="prefix
-			joint_x joint_y joint_z joint_roll joint_pitch joint_yaw
 			box_x box_y box_z
 			update_rate
@@ -9,4 +8,5 @@
 			topic_name
 			frame_name
+			*plate_name
 			">
 		<!-- Bumper Link -->
@@ -33,5 +33,6 @@
 		<joint name="${prefix}_joint" type="fixed">
 			<axis xyz="0 1 0" />
-			<origin xyz="${joint_x} ${joint_y} ${joint_z}" rpy="${joint_roll} ${joint_pitch} ${joint_yaw}"/>
+			<xacro:insert_block name="plate_name" />
+			<!--	<origin xyz="${joint_x} ${joint_y} ${joint_z}" rpy="${joint_roll} ${joint_pitch} ${joint_yaw}"/> -->
 			<parent link="${parent_link}"/>
 			<child link="${prefix}_link"/>

File: evarobot_description/urdf/evarobot_infrared.urdf.xacro (robot description, xacro)
@@ -3,5 +3,4 @@
 	<xacro:macro name="evarobot_infrared"
 		params="prefix
-				joint_x joint_y joint_z joint_roll joint_pitch joint_yaw
 				parent_link
 				scan_samples scan_resolution min_angle max_angle
@@ -9,8 +8,10 @@
 				topic_name frame_name
 				update_rate
+				*plate_name
 				">
 		<joint name="${prefix}_joint" type="fixed">
 				<axis xyz="1 0 0"/>
-				<origin xyz="${joint_x} ${joint_y} ${joint_z}" rpy="${joint_roll} ${joint_pitch} ${joint_yaw}"/>
+				<!--<origin xyz="${joint_x} ${joint_y} ${joint_z}" rpy="${joint_roll} ${joint_pitch} ${joint_yaw}"/>-->
+				<xacro:insert_block name="plate_name" />
 				<parent link="${parent_link}"/>
 				<child link="${prefix}_link"/>
@@ -25,5 +26,5 @@
 				<origin xyz="0 0 0" rpy="0 0 0" />
 				<geometry>
-					<mesh filename="package://evarobot_description/meshes/sonar_sensor/max_sonar_ez4.dae"/>
+					<mesh filename="package://evarobot_description/meshes/infrared.stl" scale="0.01 0.01 0.01"/>
 				</geometry>
 			</visual>
@@ -63,5 +64,5 @@
 				<always_on>1</always_on>
 				<update_rate>${update_rate}</update_rate>
-				<visualize>false</visualize>
+				<visualize>true</visualize>
 			</sensor>
 		</gazebo>

File: evarobot_description/urdf/evarobot_lidar.urdf.xacro (robot description, xacro)
@@ -17,5 +17,5 @@
 				<origin xyz="0 0 0" rpy="0 0 0"/>
 				<geometry>
-					<mesh filename="package://evarobot_description/meshes/hokuyo.dae"/>
+					<mesh filename="package://evarobot_description/meshes/rplidar.stl" scale="0.01 0.01 0.01" />
 				</geometry>
 			</visual>
@@ -35,5 +35,5 @@
 			<sensor type="gpu_ray" name="head_hokuyo_sensor">
 				<pose>0 0 0 0 0 0</pose>
-				<visualize>false</visualize>
+				<visualize>true</visualize>
 				<update_rate>${update_rate}</update_rate>
 				<ray>

File: evarobot_description/urdf/evarobot_sonar.urdf.xacro (robot description, xacro)
@@ -3,5 +3,4 @@
 	<xacro:macro name="evarobot_sonar"
 	params="prefix
-			joint_x joint_y joint_z joint_roll joint_pitch joint_yaw
 			parent_link
 			scan_samples scan_resolution min_angle max_angle
@@ -9,4 +8,5 @@
 			topic_name frame_name
 			update_rate
+			*plate_name
 			">
 		<link name="${prefix}_link">
@@ -19,5 +19,5 @@
 				<origin xyz="0 0 0" rpy="0 0 0" />
 				<geometry>
-					<mesh filename="package://evarobot_description/meshes/sonar_sensor/max_sonar_ez4.dae"/>
+					<mesh filename="package://evarobot_description/meshes/smo13.stl" scale="0.01 0.01 0.01"/>
 				</geometry>
 			</visual>
@@ -31,5 +31,6 @@
 		<joint name="${prefix}_joint" type="fixed">
 			<axis xyz="1 0 0" />
-			<origin xyz="${joint_x} ${joint_y} ${joint_z}" rpy="${joint_roll} ${joint_pitch} ${joint_yaw}"/>
+			<xacro:insert_block name="plate_name" />
+			<!--<origin xyz="${joint_x} ${joint_y} ${joint_z}" rpy="${joint_roll} ${joint_pitch} ${joint_yaw}"/>-->
 			<parent link="${parent_link}"/>
 			<child link="${prefix}_link"/>
@@ -64,5 +65,5 @@
 				<always_on>1</always_on>
 				<update_rate>${update_rate}</update_rate>
-				<visualize>false</visualize>
+				<visualize>true</visualize>
 			</sensor>
 		</gazebo>

File: evarobot_description/urdf/evarobot_wheel.urdf.xacro (robot description, xacro)
@@ -9,7 +9,6 @@
 				</geometry>
 			</collision>
-			<!--
 			<visual>
-				<origin rpy="0 -1.57075 0" xyz="0 0 +0.01"/>
+				<origin rpy="1.57075 0 0" xyz="0 0 0"/>
 				<geometry>
 					<cylinder length="${cylinder_length}" radius="${cylinder_radius}"/>
@@ -18,5 +17,4 @@
 				<material name="black"/>
 			</visual>
-			-->
 			<inertial>
 				<origin xyz="0 0 0" rpy="0 0 0"/>
