Commit message: added eva50 gazebo model

File: evarobot_description/urdf/evarobot.urdf.xacro (robot description, xacro)
@@ -47,6 +47,6 @@
 					   mesh_pitch="0.0"
 					   mesh_yaw="0"
-					   box_x="0.426"
-					   box_y="0.335"
+					   box_x="0.40"
+					   box_y="0.30"
 					   box_z="0.30" />
   <!-- Left Wheel -->
@@ -75,7 +75,7 @@
   <xacro:evarobot_caster prefix="front_caster"
 						 radius="0.025"
-						 x="0.153"
+						 x="0.1604"
 						 y="0.0"
-						 z="-0.225"
+						 z="-0.228"
 						 roll="-1.57075"
 						 pitch="0.0"
@@ -87,7 +87,7 @@
     <xacro:evarobot_caster prefix="rear_caster"
 						 radius="0.025"
-						 x="-0.153"
+						 x="-0.1604"
 						 y="0.0"
-						 z="-0.225"
+						 z="-0.228"
 						 roll="-1.57075"
 						 pitch="0.0"
@@ -122,7 +122,7 @@
 						 joint_y="0.0"
 						 joint_z="0.16"
-						 joint_roll="-1.57"
+						 joint_roll="0"
 						 joint_pitch="0.0"
-						 joint_yaw="-1.57"
+						 joint_yaw="0"
 						 parent_link="base_link"
 						 base_line="0.2"

File: evarobot_description/urdf/evarobot_base.urdf.xacro (robot description, xacro)
@@ -4,8 +4,9 @@
 		<link name="${prefix}_link">
 			<collision>
-				<origin xyz="${mesh_x} ${mesh_y} ${mesh_z}" rpy="${mesh_roll} ${mesh_pitch} ${mesh_yaw}" />
+				<origin xyz="0 0 0" rpy="0 0 0"/>
+				<!--<origin xyz="${mesh_x} ${mesh_y} ${mesh_z}" rpy="${mesh_roll} ${mesh_pitch} ${mesh_yaw}" /> -->
 				<geometry>
-					<mesh filename="package://evarobot_description/meshes/eva50.stl" scale="0.01 0.01 0.01"/>
-<!--				<box size="${box_x} ${box_y} ${box_z}"/> -->
+<!--					<mesh filename="package://evarobot_description/meshes/eva50.stl" scale="0.01 0.01 0.01"/>   -->
+				<box size="${box_x} ${box_y} ${box_z}"/>
 				</geometry>
 			</collision>

File: evarobot_description/urdf/evarobot_caster.urdf.xacro (robot description, xacro)
@@ -19,6 +19,6 @@
 			<inertial>
 				<origin xyz="0 0 0" rpy="0 0 0"/>
-				<mass value="5"/>
-				<inertia ixx="1e-6" ixy="0" ixz="0" iyy="1e-6" iyz="0" izz="1e-6" />
+				<mass value="0.5"/>
+				<inertia ixx="1e-1" ixy="0" ixz="0" iyy="1e-1" iyz="0" izz="1e-1" />
 			</inertial>
 		</link>
@@ -32,6 +32,6 @@
 			<origin rpy="${roll} ${pitch} ${yaw}" xyz="${x} ${y} ${z}"/>
 			<axis xyz="${axis_x} ${axis_y} ${axis_z}"/>
-			<limit effort="100" velocity="100"/>
-			<joint_properties damping="0.0" friction="0.0"/>
+			<limit effort="10" velocity="10"/>
+			<joint_properties damping="0.0" friction="0.3"/>
 		</joint>
 	</xacro:macro>

File: evarobot_description/urdf/evarobot_infrared.urdf.xacro (robot description, xacro)
@@ -23,4 +23,5 @@
 				<inertia ixx="0.000000017" ixy="0" ixz="0" iyy="0.000000017" iyz="0" izz="0.000000017" />
 			</inertial>
+<!--
 			<visual>
 				<origin xyz="0 0 0" rpy="0 0 0" />
@@ -29,4 +30,5 @@
 				</geometry>
 			</visual>
+	-->
 			<collision>
 				<origin xyz="0 0 0" rpy="0 0 0" />

File: evarobot_description/urdf/evarobot_kinect.urdf.xacro (robot description, xacro)
@@ -9,5 +9,5 @@
 			">
 		<!-- Kinect Link -->
-		<link name="kinect_dummy">
+		<link name="${prefix}_link">
 			<collision>
 				<origin xyz="0 0 0" rpy="0 0 0"/>
@@ -31,17 +31,17 @@
 		<joint name="${prefix}_joint" type="fixed">
 			<axis xyz="0 1 0" />
-			<origin xyz="${joint_x} ${joint_y} ${joint_z}" rpy="0 0 0"/>
+			<origin xyz="${joint_x} ${joint_y} ${joint_z}" rpy="${joint_roll} ${joint_pitch} ${joint_yaw}"/>
 			<parent link="${parent_link}"/>
-			<child link="kinect_dummy"/>
+			<child link="${prefix}_link"/>
 		</joint>
 		<!-- Kinect Dummy Link -->
-		<link name="${prefix}_link">
+		<link name="kinect_dummy">
 			<pose>0 0 0 0 0 0</pose>
 		</link>
 		<!-- Kinect Dummy Joint -->
 		<joint name="kinect_joint_dummy" type="fixed">
-			<origin xyz="0 0 0" rpy="${joint_roll} ${joint_pitch} ${joint_yaw}"/>
-			<parent link="kinect_dummy"/>
-			<child link="${prefix}_link"/>
+			<origin xyz="0 0 0" rpy="-1.57 0.0 -1.57"/>
+			<parent link="${prefix}_link"/>
+			<child link="kinect_dummy"/>
 			<axis xyz="0 1 0"/>
 		</joint>

File: evarobot_description/urdf/evarobot_lidar.urdf.xacro (robot description, xacro)
@@ -14,5 +14,5 @@
 				</geometry>
 			</collision>
-			<visual>
+<!--			<visual>
 				<origin xyz="0 0 0" rpy="0 0 0"/>
 				<geometry>
@@ -20,4 +20,5 @@
 				</geometry>
 			</visual>
+-->
 			<inertial>
 				<mass value="1e-5" />

File: evarobot_description/urdf/evarobot_sonar.urdf.xacro (robot description, xacro)
@@ -16,5 +16,5 @@
 				<inertia ixx="0.000000017" ixy="0" ixz="0" iyy="0.000000017" iyz="0" izz="0.000000017" />
 			</inertial>
-			<visual>
+<!--			<visual>
 				<origin xyz="0 0 0" rpy="0 0 0" />
 				<geometry>
@@ -22,4 +22,5 @@
 				</geometry>
 			</visual>
+-->
 			<collision>
 				<origin xyz="0 0 0" rpy="0 0 0" />

Commit message: modified placement of sonar and infrared sensors

File: evarobot_description/urdf/evarobot.urdf.xacro (robot description, xacro)
@@ -177,18 +177,18 @@
 	-->
   <!-- Sonar -->
-  <xacro:evarobot_sonar prefix="sensor/sonar0"
-						parent_link="base_link"
-						scan_samples="320"
-						scan_resolution="1"
-						min_angle="-0.479965544"
-						max_angle="0.479965544"
-						range_resolution="0.01"
-						min_range="0.02"
-						max_range="5.0"
-						topic_name="sonar0"
-						frame_name="sensor/sonar0_link"
-						update_rate="4">
-						  <origin xyz="0.045 -0.168 0.03" rpy="0 0 ${-pi/2}" />
-  </xacro:evarobot_sonar>
+	<xacro:evarobot_sonar prefix="sensor/sonar0"
+				parent_link="base_link"
+				scan_samples="320"
+				scan_resolution="1"
+				min_angle="-0.479965544"
+				max_angle="0.479965544"
+				range_resolution="0.01"
+				min_range="0.02"
+				max_range="5.0"
+				topic_name="sonar0"
+				frame_name="sensor/sonar0_link"
+				update_rate="4" >
+				<origin xyz="0.130 -0.147 0.03" rpy="0 0 ${-pi/3}" />
+	</xacro:evarobot_sonar>
   <xacro:evarobot_sonar prefix="sensor/sonar1"
 						parent_link="base_link"
@@ -205,5 +205,61 @@
 								<origin xyz="0.213 0.0 0.03" rpy="0 0 0" />
 	</xacro:evarobot_sonar>
-  <xacro:evarobot_sonar prefix="sensor/sonar2"
+	<xacro:evarobot_sonar prefix="sensor/sonar2"
+				parent_link="base_link"
+				scan_samples="320"
+				scan_resolution="1"
+				min_angle="-0.479965544"
+				max_angle="0.479965544"
+				range_resolution="0.01"
+				min_range="0.02"
+				max_range="5.0"
+				topic_name="sonar2"
+				frame_name="sensor/sonar2_link"
+				update_rate="4" >
+				<origin xyz="0.130 0.147 0.03" rpy="0 0 ${pi/3}" />
+	</xacro:evarobot_sonar>
+	<xacro:evarobot_sonar prefix="sensor/sonar3"
+					parent_link="base_link"
+					scan_samples="320"
+					scan_resolution="1"
+					min_angle="-0.479965544"
+					max_angle="0.479965544"
+					range_resolution="0.01"
+					min_range="0.02"
+					max_range="5.0"
+					topic_name="sonar3"
+					frame_name="sensor/sonar3_link"
+					update_rate="4">
+						<origin xyz="-0.045 0.168 0.03" rpy="0 0 ${pi/2}" />
+	</xacro:evarobot_sonar>
+	<xacro:evarobot_sonar prefix="sensor/sonar4"
+					parent_link="base_link"
+					scan_samples="320"
+					scan_resolution="1"
+					min_angle="-0.479965544"
+					max_angle="0.479965544"
+					range_resolution="0.01"
+					min_range="0.02"
+					max_range="5.0"
+					topic_name="sonar4"
+					frame_name="sensor/sonar4_link"
+					update_rate="4" >
+					<origin xyz="-0.191 0.084 0.03" rpy="0 0 ${5*pi/6}" />
+	</xacro:evarobot_sonar>
+	<xacro:evarobot_sonar prefix="sensor/sonar5"
+					parent_link="base_link"
+					scan_samples="320"
+					scan_resolution="1"
+					min_angle="-0.479965544"
+					max_angle="0.479965544"
+					range_resolution="0.01"
+					min_range="0.02"
+					max_range="5.0"
+					topic_name="sonar5"
+					frame_name="sensor/sonar5_link"
+					update_rate="4" >
+					<origin xyz="-0.191 -0.084 0.03" rpy="0 0 ${-5*pi/6}" />
+	</xacro:evarobot_sonar>
+  <xacro:evarobot_sonar prefix="sensor/sonar6"
 						parent_link="base_link"
 						scan_samples="320"
@@ -214,37 +270,9 @@
 						min_range="0.02"
 						max_range="5.0"
-						topic_name="sonar2"
-						frame_name="sensor/sonar2_link"
+						topic_name="sonar6"
+						frame_name="sensor/sonar6_link"
 						update_rate="4">
-						  <origin xyz="0.045 0.168 0.03" rpy="0 0 ${pi/2}" />
-	</xacro:evarobot_sonar>
-  <xacro:evarobot_sonar prefix="sensor/sonar3"
-						parent_link="base_link"
-						scan_samples="320"
-						scan_resolution="1"
-						min_angle="-0.479965544"
-						max_angle="0.479965544"
-						range_resolution="0.01"
-						min_range="0.02"
-						max_range="5.0"
-						topic_name="sonar3"
-						frame_name="sensor/sonar3_link"
-						update_rate="4" >
-						  <origin xyz="-0.191 0.084 0.03" rpy="0 0 ${5*pi/6}" />
-	</xacro:evarobot_sonar>
-	  <xacro:evarobot_sonar prefix="sensor/sonar4"
-						parent_link="base_link"
-						scan_samples="320"
-						scan_resolution="1"
-						min_angle="-0.479965544"
-						max_angle="0.479965544"
-						range_resolution="0.01"
-						min_range="0.02"
-						max_range="5.0"
-						topic_name="sonar4"
-						frame_name="sensor/sonar4_link"
-						update_rate="4" >
-  <origin xyz="-0.191 -0.084 0.03" rpy="0 0 ${-5*pi/6}" />
-	</xacro:evarobot_sonar>
+						  <origin xyz="-0.045 -0.168 0.03" rpy="0 0 ${-pi/2}" />
+  </xacro:evarobot_sonar>
   <!-- Infrared -->
   <xacro:evarobot_infrared prefix="sensor/ir0"
@@ -260,5 +288,5 @@
 						   frame_name="sensor/ir0_link"
 						   update_rate="4" >
-						   	     <origin xyz="0.191 -0.084 0.03" rpy="0 0 ${-pi/6}" />
+						   	     <origin xyz="0.191 -0.084 -0.122" rpy="0 0 ${-pi/6}" />
 	</xacro:evarobot_infrared>
   <xacro:evarobot_infrared prefix="sensor/ir1"
@@ -274,5 +302,5 @@
 						   frame_name="sensor/ir1_link"
 						   update_rate="4">
-						   		<origin xyz="0.191 0.084 0.03" rpy="0 0 ${pi/6}" />
+						   		<origin xyz="0.191 0.084 -0.122" rpy="0 0 ${pi/6}" />
 	</xacro:evarobot_infrared>
   <xacro:evarobot_infrared prefix="sensor/ir2"
@@ -288,5 +316,5 @@
 						   frame_name="sensor/ir2_link"
 						   update_rate="4">
-						   		<origin xyz="-0.045 0.168 0.03" rpy="0 0 ${pi/2}" />
+						   		<origin xyz="-0.130 0.147 -0.122" rpy="0 0 ${2*pi/3}" />
 	</xacro:evarobot_infrared>
   <xacro:evarobot_infrared prefix="sensor/ir3"
@@ -302,5 +330,5 @@
 						   frame_name="sensor/ir3_link"
 						   update_rate="4">
-						   	    <origin xyz="-0.045 -0.168 0.03" rpy="0 0 ${-pi/2}" />
+						   	    <origin xyz="-0.130 -0.147 -0.122" rpy="0 0 ${-2*pi/3}" />
 	</xacro:evarobot_infrared>
 </robot>

Commit message: modified sensors in gazebo model

File: evarobot_description/urdf/evarobot.urdf.xacro (robot description, xacro)
@@ -104,5 +104,5 @@
                         joint_roll="0.0"
                         joint_pitch="0.0"
-                        joint_yaw="-1.5708"
+                        joint_yaw="3.14"
 												update_rate="40"
 												samples="720"
@@ -117,4 +117,5 @@
 												topic_name="lidar"
 												frame_name="lidar_link" />
+<!-- joint_yaw="-1.5708" -->
   <!-- Kinect -->
    <xacro:evarobot_kinect prefix="sensor/kinect"
@@ -176,5 +177,5 @@
 					   robot_namespace="evarobot" />
 	-->
-  <!-- Sonar -->
+ <!-- Sonar -->
 	<xacro:evarobot_sonar prefix="sensor/sonar0"
 				parent_link="base_link"

File: evarobot_description/urdf/evarobot_wheel.urdf.xacro (robot description, xacro)
@@ -13,5 +13,5 @@
 				<geometry>
 					<cylinder length="${cylinder_length}" radius="${cylinder_radius}"/>
-					<mesh filename="package://evarobot_description/meshes/wheel.stl" scale="0.001 0.001 0.001"/>
+					<mesh filename="model://evarobot/meshes/wheel.stl" scale="0.001 0.001 0.001"/>
 				</geometry>
 				<material name="black"/>
