Commit message: modify robot model for new mesh files

File: evarobot_description/urdf/evarobot.urdf.xacro (robot description, xacro)
@@ -6,4 +6,5 @@
   <xacro:property name="pi" value="3.1415926535897931" />
   <!-- Includes -->
+  <xacro:include filename="$(find evarobot_description)/urdf/materials.urdf.xacro"/>
   <xacro:include filename="$(find evarobot_description)/urdf/evarobot_base.urdf.xacro"/>
   <xacro:include filename="$(find evarobot_description)/urdf/evarobot_caster.urdf.xacro"/>
@@ -25,5 +26,4 @@
 		<publishWheelJointState>true</publishWheelJointState>
 		<wheelAcceleration>1</wheelAcceleration>
-	  <!--  Plugin arkadan suruslu robotlar icin yapildigindan jointler ters yazildi  -->
 	  <leftJoint>right_wheel_joint</leftJoint>
 	  <rightJoint>left_wheel_joint</rightJoint>
@@ -43,5 +43,5 @@
 					   mesh_x="0.065"
 					   mesh_y="-0.11"
-					   mesh_z="-0.20"
+					   mesh_z="-0.15"
 					   mesh_roll="0.0"
 					   mesh_pitch="0.0"
@@ -54,5 +54,5 @@
 						joint_x="0.0"
 						joint_y="0.16"
-						joint_z="-0.1685"
+						joint_z="${-0.15 + (85-54)/1000}"
 						joint_roll="0.0"
 						joint_pitch="0.0"
@@ -65,5 +65,5 @@
 						joint_x="0.0"
 						joint_y="-0.16"
-						joint_z="-0.1685"
+						joint_z="${-0.15 + (85-54)/1000}"
 						joint_roll="0.0"
 						joint_pitch="0.0"
@@ -77,6 +77,6 @@
 						 x="0.1604"
 						 y="0.0"
-						 z="-0.228"
-						 roll="-1.57075"
+						 z="${-0.15 -13.5/2000}"
+						 roll="0.0"
 						 pitch="0.0"
 						 yaw="0.0"
@@ -89,6 +89,6 @@
 						 x="-0.1604"
 						 y="0.0"
-						 z="-0.228"
-						 roll="-1.57075"
+						 z="${-0.15 -13.5/2000}"
+						 roll="0.0"
 						 pitch="0.0"
 						 yaw="0.0"
@@ -101,5 +101,5 @@
                         joint_x="-0.15"
                         joint_y="0.0"
-                        joint_z="0.4415"
+                        joint_z="${0.4415 + 100/1000}"
                         joint_roll="0.0"
                         joint_pitch="0.0"
@@ -117,49 +117,16 @@
 												topic_name="lidar"
 												frame_name="lidar_link" />
-<!-- joint_yaw="-1.5708" -->
   <!-- Kinect -->
    <xacro:evarobot_kinect prefix="kinect"
 						 joint_x="0.17"
 						 joint_y="0.0"
-						 joint_z="0.16"
-						 joint_roll="0"
+						 joint_z="${0.21 - 18.7/1000}"
+						 joint_roll="0.0"
 						 joint_pitch="0.0"
-						 joint_yaw="0"
+						 joint_yaw="0.0"
 						 parent_link="base_link"
 						 base_line="0.2"
 						 update_rate="1.0"
 						 camera_name="camera" />
-  <!-- Bumper -->
-  <xacro:evarobot_bumper prefix="bumper0"
-						 box_x="0.015"
-						 box_y="0.015"
-						 box_z="0.020"
-						 update_rate="10.0"
-						 parent_link="base_link"
-						 topic_name="bumper0"
-						 frame_name="bumper0_link" >
-  <origin xyz="0.191 -0.084 -0.122" rpy="0 0 ${-pi/6}" />
-						 </xacro:evarobot_bumper>
-  <xacro:evarobot_bumper prefix="bumper1"
-						 box_x="0.015"
-						 box_y="0.015"
-						 box_z="0.020"
-						 update_rate="10.0"
-						 parent_link="base_link"
-						 topic_name="bumper1"
-						 frame_name="bumper1_link" >
-						   <origin xyz="0.213 0.0 -0.122" rpy="0 0 0" />
-  <origin xyz="0.213 0.0 -0.122" rpy="0 0 0" />
-						</xacro:evarobot_bumper>
-  <xacro:evarobot_bumper prefix="bumper2"
-						 box_x="0.015"
-						 box_y="0.015"
-						 box_z="0.020"
-						 update_rate="10.0"
-						 parent_link="base_link"
-						 topic_name="bumper2"
-						 frame_name="bumper2_link" >
-  <origin xyz="0.191 0.084 -0.122" rpy="0 0 ${pi/6}" />
-						 </xacro:evarobot_bumper>
   <!-- AHRS/IMU -->
   <xacro:evarobot_ahrs prefix="imu"
@@ -189,5 +156,5 @@
 				frame_name="sonar0_link"
 				update_rate="4" >
-				<origin xyz="0.130 -0.147 0.03" rpy="0 0 ${-pi/3}" />
+				<origin xyz="0.130 -0.147 ${0.03+50/1000}" rpy="0 0 ${-pi/3}" />
 	</xacro:evarobot_sonar>
   <xacro:evarobot_sonar prefix="sonar1"
@@ -203,5 +170,5 @@
 						frame_name="sonar1_link"
 						update_rate="4">
-								<origin xyz="0.213 0.0 0.03" rpy="0 0 0" />
+								<origin xyz="0.213 0.0 ${0.03+50/1000}" rpy="0 0 0" />
 	</xacro:evarobot_sonar>
 	<xacro:evarobot_sonar prefix="sonar2"
@@ -217,5 +184,5 @@
 				frame_name="sonar2_link"
 				update_rate="4" >
-				<origin xyz="0.130 0.147 0.03" rpy="0 0 ${pi/3}" />
+				<origin xyz="0.130 0.147 ${0.03+50/1000}" rpy="0 0 ${pi/3}" />
 	</xacro:evarobot_sonar>
 	<xacro:evarobot_sonar prefix="sonar3"
@@ -231,5 +198,5 @@
 					frame_name="sonar3_link"
 					update_rate="4">
-						<origin xyz="-0.045 0.168 0.03" rpy="0 0 ${pi/2}" />
+						<origin xyz="-0.045 0.168 ${0.03+50/1000}" rpy="0 0 ${pi/2}" />
 	</xacro:evarobot_sonar>
 	<xacro:evarobot_sonar prefix="sonar4"
@@ -245,5 +212,5 @@
 					frame_name="sonar4_link"
 					update_rate="4" >
-					<origin xyz="-0.191 0.084 0.03" rpy="0 0 ${5*pi/6}" />
+					<origin xyz="-0.191 0.084 ${0.03+50/1000}" rpy="0 0 ${5*pi/6}" />
 	</xacro:evarobot_sonar>
 	<xacro:evarobot_sonar prefix="sonar5"
@@ -259,5 +226,5 @@
 					frame_name="sonar5_link"
 					update_rate="4" >
-					<origin xyz="-0.191 -0.084 0.03" rpy="0 0 ${-5*pi/6}" />
+					<origin xyz="-0.191 -0.084 ${0.03+50/1000}" rpy="0 0 ${-5*pi/6}" />
 	</xacro:evarobot_sonar>
   <xacro:evarobot_sonar prefix="sonar6"
@@ -273,5 +240,5 @@
 						frame_name="sonar6_link"
 						update_rate="4">
-						  <origin xyz="-0.045 -0.168 0.03" rpy="0 0 ${-pi/2}" />
+						  <origin xyz="-0.045 -0.168 ${0.03+50/1000}" rpy="0 0 ${-pi/2}" />
   </xacro:evarobot_sonar>
   <!-- Infrared -->
@@ -288,5 +255,5 @@
 						   frame_name="ir0_link"
 						   update_rate="4" >
-						   	     <origin xyz="0.191 -0.084 -0.122" rpy="0 0 ${-pi/6}" />
+						   	     <origin xyz="0.191 -0.084 ${-0.122+50/1000}" rpy="0 0 ${-pi/6}" />
 	</xacro:evarobot_infrared>
   <xacro:evarobot_infrared prefix="ir1"
@@ -302,5 +269,5 @@
 						   frame_name="ir1_link"
 						   update_rate="4">
-						   		<origin xyz="0.191 0.084 -0.122" rpy="0 0 ${pi/6}" />
+						   		<origin xyz="0.191 0.084 ${-0.122+50/1000}" rpy="0 0 ${pi/6}" />
 	</xacro:evarobot_infrared>
   <xacro:evarobot_infrared prefix="ir2"
@@ -316,5 +283,5 @@
 						   frame_name="ir2_link"
 						   update_rate="4">
-						   		<origin xyz="-0.130 0.147 -0.122" rpy="0 0 ${2*pi/3}" />
+						   		<origin xyz="-0.130 0.147 ${-0.122+50/1000}" rpy="0 0 ${2*pi/3}" />
 	</xacro:evarobot_infrared>
   <xacro:evarobot_infrared prefix="ir3"
@@ -330,5 +297,36 @@
 						   frame_name="ir3_link"
 						   update_rate="4">
-						   	    <origin xyz="-0.130 -0.147 -0.122" rpy="0 0 ${-2*pi/3}" />
+						   	    <origin xyz="-0.130 -0.147 ${-0.122+50/1000}" rpy="0 0 ${-2*pi/3}" />
 	</xacro:evarobot_infrared>
+ <!-- Bumper -->
+  <xacro:evarobot_bumper prefix="bumper0"
+						 box_x="0.015"
+						 box_y="0.015"
+						 box_z="0.020"
+						 update_rate="10.0"
+						 parent_link="base_link"
+						 topic_name="bumper0"
+						 frame_name="bumper0_link" >
+  <origin xyz="0.191 -0.084 ${-0.122+50/1000}" rpy="0 0 ${-pi/6}" />
+						 </xacro:evarobot_bumper>
+  <xacro:evarobot_bumper prefix="bumper1"
+						 box_x="0.015"
+						 box_y="0.015"
+						 box_z="0.020"
+						 update_rate="10.0"
+						 parent_link="base_link"
+						 topic_name="bumper1"
+						 frame_name="bumper1_link" >
+						   <origin xyz="0.213 0.0 ${-0.122+50/1000}" rpy="0 0 0" />
+						</xacro:evarobot_bumper>
+  <xacro:evarobot_bumper prefix="bumper2"
+						 box_x="0.015"
+						 box_y="0.015"
+						 box_z="0.020"
+						 update_rate="10.0"
+						 parent_link="base_link"
+						 topic_name="bumper2"
+						 frame_name="bumper2_link" >
+  <origin xyz="0.191 0.084 ${-0.122+50/1000}" rpy="0 0 ${pi/6}" />
+						 </xacro:evarobot_bumper>
 </robot>

File: evarobot_description/urdf/evarobot_ahrs.urdf.xacro (robot description, xacro)
@@ -6,5 +6,5 @@
 				<mass value="0.001"/>
 				<origin rpy="0 0 0" xyz="0 0 0"/>
-				<inertia ixx="0.0001" ixy="0" ixz="0" iyy="0.000001" iyz="0" izz="0.0001"/>
+				<inertia ixx="0.0001" ixy="0" ixz="0" iyy="0.0001" iyz="0" izz="0.0001"/>
 			</inertial>
 			<visual>

File: evarobot_description/urdf/evarobot_base.urdf.xacro (robot description, xacro)
@@ -5,8 +5,6 @@
 			<collision>
 				<origin xyz="0 0 0" rpy="0 0 0"/>
-				<!--<origin xyz="${mesh_x} ${mesh_y} ${mesh_z}" rpy="${mesh_roll} ${mesh_pitch} ${mesh_yaw}" /> -->
 				<geometry>
-<!--					<mesh filename="package://evarobot_description/meshes/eva50.stl" scale="0.01 0.01 0.01"/>   -->
-				<box size="${box_x} ${box_y} ${box_z}"/>
+					<box size="${box_x} ${box_y} ${box_z}"/>
 				</geometry>
 			</collision>
@@ -14,20 +12,52 @@
 				<origin xyz="${mesh_x} ${mesh_y} ${mesh_z}" rpy="${mesh_roll} ${mesh_pitch} ${mesh_yaw}" />
 				<geometry>
-				<!-- <box size="${box_x} ${box_y} ${box_z}"/> -->
-				<mesh filename="package://evarobot_description/meshes/eva50.dae" scale="0.01 0.01 0.01"/>
+					<mesh filename="package://evarobot_description/meshes/base.stl" scale="1 1 1"/>
 				</geometry>
-				<material name="red">
-					<color rgba="0.4 0.7 .8 1"/>
-				</material>
+				<material name="Black" />
 			</visual>
 			<inertial>
 				<origin xyz="0 0 0" rpy="0 0 0"/>
-				<mass value="15"/>
+				<mass value="10.0"/>
 				<inertia
-					ixx="0.875" ixy="0.155" ixz="0.143"
-					iyy="0.155" iyz="0.143"
-					izz="0.143"/>
+					ixx="1.0" ixy="0" ixz="0"
+					iyy="1.0" iyz="0"
+					izz="1.0"/>
 			</inertial>
 		</link>
+		<gazebo reference="${prefix}_link">
+      <material>Gazebo/Black</material>
+		</gazebo>
+		<link name="${prefix}color_link">
+			<collision>
+				<origin xyz="0 0 0" rpy="0 0 0"/>
+				<geometry>
+					<box size="0.0001 0.0001 0.0001"/>
+				</geometry>
+			</collision>
+			<visual>
+				<origin xyz="${mesh_x} ${mesh_y} ${mesh_z}" rpy="${mesh_roll} ${mesh_pitch} ${mesh_yaw}" />
+				<geometry>
+					<mesh filename="package://evarobot_description/meshes/base_orange.stl" scale="1 1 1"/>
+				</geometry>
+				<material name="Orange" />
+			</visual>
+			<inertial>
+				<origin xyz="0 0 0" rpy="0 0 0"/>
+				<mass value="0.0001"/>
+				<inertia
+					ixx="1e-6" ixy="0.0" ixz="0.0"
+					iyy="1e-6" iyz="0.0"
+					izz="1e-6"/>
+			</inertial>
+		</link>
+		<gazebo reference="${prefix}color_link">
+      <material>Gazebo/Orange</material>
+		</gazebo>
+		<joint name="${prefix}color_joint" type="fixed">
+			<axis xyz="0 1 0" />
+			<origin xyz="0 0 0" rpy="0 0 0"/>
+			<parent link="${prefix}_link"/>
+			<child link="${prefix}color_link"/>
+		</joint>
 	</xacro:macro>
 </robot>

File: evarobot_description/urdf/evarobot_kinect.urdf.xacro (robot description, xacro)
@@ -8,75 +8,113 @@
 			camera_name
 			">
-		<!-- Kinect Link -->
-		<link name="${prefix}_link">
-			<collision>
-				<origin xyz="0 0 0" rpy="0 0 0"/>
-				<geometry>
-					<box size="0.1 0.1 0.1"/>
-				</geometry>
-			</collision>
-			<visual>
-				<origin xyz="0 0 0" rpy="0 0 0"/>
-				<geometry>
-					<mesh filename="package://evarobot_description/meshes/kinect.dae"/>
-				</geometry>
-			</visual>
-			<inertial>
-				<mass value="1e-5" />
-				<origin xyz="0 0 0" rpy="0 0 0"/>
-				<inertia ixx="1e-6" ixy="0" ixz="0" iyy="1e-6" iyz="0" izz="1e-6" />
-			</inertial>
-		</link>
-		<!-- Kinect Joint -->
-		<joint name="${prefix}_joint" type="fixed">
-			<axis xyz="0 1 0" />
+    <joint name="camera_rgb_joint" type="fixed">
+			<origin xyz="0.0 -0.02 0.0" rpy="0.0 0.0 0.0"/>
+			<parent link="camera_link"/>
+      <child link="camera_rgb_frame" />
+    </joint>
+    <link name="camera_rgb_frame"/>
+    <joint name="camera_rgb_optical_joint" type="fixed">
+      <origin xyz="0 0 0" rpy="${-pi/2} 0 ${-pi/2}" />
+      <parent link="camera_rgb_frame" />
+      <child link="camera_rgb_optical_frame" />
+    </joint>
+    <link name="camera_rgb_optical_frame"/>
+    <joint name="camera_joint" type="fixed">
 			<origin xyz="${joint_x} ${joint_y} ${joint_z}" rpy="${joint_roll} ${joint_pitch} ${joint_yaw}"/>
-			<parent link="${parent_link}"/>
-			<child link="${prefix}_link"/>
-		</joint>
-		<!-- Kinect Dummy Link -->
-		<link name="kinect_dummy">
-			<pose>0 0 0 0 0 0</pose>
-		</link>
-		<!-- Kinect Dummy Joint -->
-		<joint name="kinect_joint_dummy" type="fixed">
-			<origin xyz="0 0 0" rpy="-1.57 0.0 -1.57"/>
-			<parent link="${prefix}_link"/>
-			<child link="kinect_dummy"/>
-			<axis xyz="0 1 0"/>
-		</joint>
-		<!-- Kinect Gazebo Plugin -->
-		<gazebo reference="${prefix}_link">
-			<sensor type="depth" name="openni_camera_camera">
-				<always_on>1</always_on>
-				<visualize>false</visualize>
-				<camera>
-					<horizontal_fov>1.047</horizontal_fov>
-					<image>
-						<width>640</width>
-						<height>480</height>
-						<format>R8G8B8</format>
-					</image>
-					<depth_camera>
-					</depth_camera>
-					<clip>
-						<near>0.2</near>
-						<far>100</far>
-					</clip>
-				</camera>
-				<plugin name="${prefix}_controller" filename="libgazebo_ros_openni_kinect.so">
-					<baseline>${base_line}</baseline>
-					<alwaysOn>true</alwaysOn>
-					<updateRate>${update_rate}</updateRate>
-					<cameraName>${camera_name}</cameraName>
-					<imageTopicName>rgb/image_raw</imageTopicName>
-					<depthImageCameraInfoTopicName>depth/image_camera_info</depthImageCameraInfoTopicName>
-					<pointCloudCutoffMax>5.0</pointCloudCutoffMax>
-					<cameraInfoTopicName>camera_info</cameraInfoTopicName>
-					<depthImageTopicName>depth/image_raw</depthImageTopicName>
-					<depthImageInfoTopicName>depth/camera_info</depthImageInfoTopicName>
-					<pointCloudTopicName>depth/points</pointCloudTopicName>
-					<frameName>kinect_dummy</frameName>
-					<pointCloudCutoff>0.5</pointCloudCutoff>
+      <parent link="${parent_link}"/>
+      <child link="camera_link"/>
+    </joint>
+    <link name="camera_link">
+      <visual>
+        <origin xyz="0.0 0.0 0.004" rpy="0 0 0"/>
+        <geometry>
+          <mesh filename="package://evarobot_description/meshes/xtion_pro_camera.dae"/>
+        </geometry>
+      </visual>
+      <collision>
+        <origin xyz="0.0 0.0 0.0" rpy="0 0 0" />
+        <geometry>
+        <box size="0.0730 0.2760 0.0720"/>
+      </geometry>
+      </collision>
+      <inertial>
+        <mass value="0.170" />
+        <origin xyz="0 0 0" />
+        <inertia ixx="0.001152600" ixy="0.0" ixz="0.0"
+                 iyy="0.000148934" iyz="0.0"
+                 izz="0.001154654" />
+      </inertial>
+    </link>
+    <joint name="camera_depth_joint" type="fixed">
+      <origin xyz="0 -0.045 0" rpy="0 0 0" />
+      <parent link="camera_link" />
+      <child link="camera_depth_frame" />
+    </joint>
+    <link name="camera_depth_frame"/>
+    <joint name="camera_depth_optical_joint" type="fixed">
+      <origin xyz="0 0 0" rpy="${-pi/2} 0 ${-pi/2}" />
+      <parent link="camera_depth_frame" />
+      <child link="camera_depth_optical_frame" />
+    </joint>
+    <link name="camera_depth_optical_frame"/>
+    <!-- Asus mount -->
+    <joint name="mount_asus_xtion_pro_joint" type="fixed">
+			<origin xyz="${0.17 -16.5/1000 + 0.015} -0.0050 ${0.21 - 18.7/1000 -35/1000}" rpy="${pi/2} 0 ${-pi/2}"/>
+      <parent link="base_link"/>
+      <child link="mount_asus_xtion_pro_link"/>
+    </joint>
+    <link name="mount_asus_xtion_pro_link">
+      <visual>
+        <origin xyz="0 0 0" rpy="0 0 0"/>
+        <geometry>
+          <mesh filename="package://evarobot_description/meshes/asus_base.stl"/>
+        </geometry>
+        <material name="Black"/>
+      </visual>
+      <collision>
+        <origin xyz="0.0 0.0 0.0" rpy="0 0 0" />
+        <geometry>
+        <box size="0.2760 0.0330 0.0120"/>
+      </geometry>
+      </collision>
+      <inertial>
+        <mass value="0.170" />
+        <origin xyz="0 0 0" />
+        <inertia ixx="0.001152600" ixy="0.0" ixz="0.0"
+                 iyy="0.000148934" iyz="0.0"
+                 izz="0.001154654" />
+      </inertial>
+    </link>
+		<gazebo reference="mount_asus_xtion_pro_link">
+			<material>Gazebo/Black</material>
+		</gazebo>
+		<gazebo reference="camera_link">
+      <sensor type="depth" name="camera">
+        <always_on>true</always_on>
+        <update_rate>20.0</update_rate>
+        <camera>
+          <horizontal_fov>${60.0*pi/180.0}</horizontal_fov>
+          <image>
+            <format>R8G8B8</format>
+            <width>640</width>
+            <height>480</height>
+          </image>
+          <clip>
+            <near>0.05</near>
+            <far>8.0</far>
+          </clip>
+        </camera>
+        <plugin name="kinect_camera_controller" filename="libgazebo_ros_openni_kinect.so">
+          <cameraName>camera</cameraName>
+          <alwaysOn>true</alwaysOn>
+          <updateRate>10</updateRate>
+          <imageTopicName>rgb/image_raw</imageTopicName>
+          <depthImageTopicName>depth/image_raw</depthImageTopicName>
+          <pointCloudTopicName>depth/points</pointCloudTopicName>
+          <cameraInfoTopicName>rgb/camera_info</cameraInfoTopicName>
+          <depthImageCameraInfoTopicName>depth/camera_info</depthImageCameraInfoTopicName>
+          <frameName>camera_depth_optical_frame</frameName>
+          <baseline>0.1</baseline>
+					<pointCloudCutoff>0.4</pointCloudCutoff>
 					<distortionK1>0.00000001</distortionK1>
 					<distortionK2>0.00000001</distortionK2>
@@ -89,7 +127,7 @@
 					<focalLength>0</focalLength>
 					<hackBaseline>0</hackBaseline>
-				</plugin>
-			</sensor>
-		</gazebo>
+        </plugin>
+      </sensor>
+    </gazebo>
 	</xacro:macro>
 </robot>

File: evarobot_description/urdf/evarobot_lidar.urdf.xacro (robot description, xacro)
@@ -14,11 +14,11 @@
 				</geometry>
 			</collision>
-<!--			<visual>
-				<origin xyz="0 0 0" rpy="0 0 0"/>
+			<visual>
+				<origin xyz="${-55/1000} ${-110/1000} ${-50/1000}" rpy="${-pi/2} ${pi} 0"/>
 				<geometry>
-					<mesh filename="package://evarobot_description/meshes/rplidar.stl" scale="0.01 0.01 0.01" />
+					<mesh filename="package://evarobot_description/meshes/rplidar.stl" scale="0.001 0.001 0.001" />
 				</geometry>
+				<material name="Black" />
 			</visual>
--->
 			<inertial>
 				<mass value="1e-5" />
@@ -34,4 +34,5 @@
 		</joint>
 		<gazebo reference="${prefix}_link">
+			<material>Gazebo/Black</material>
 			<sensor type="gpu_ray" name="head_hokuyo_sensor">
 				<pose>0 0 0 0 0 0</pose>

File: evarobot_description/urdf/evarobot_wheel.urdf.xacro (robot description, xacro)
@@ -10,17 +10,28 @@
 			</collision>
 			<visual>
-				<origin rpy="1.57075 0 0" xyz="0 0 0"/>
+				<origin rpy="0 0 ${pi/2}" xyz="0 0 0"/>
 				<geometry>
-					<cylinder length="${cylinder_length}" radius="${cylinder_radius}"/>
-					<mesh filename="model://evarobot/meshes/wheel.dae" scale="0.001 0.001 0.001"/>
+					 <mesh filename="package://evarobot_description/meshes/rim.stl" scale="1 1 1"/>
 				</geometry>
-				<material name="black"/>
+				<material name="Grey"/>
 			</visual>
 			<inertial>
-				<origin xyz="0 0 0" rpy="0 0 0"/>
-				<mass value="0.75"/>
-				<inertia ixx="1e-2" ixy="0" ixz="0" iyy="1e-2" iyz="0" izz="1e-2" />
+				<origin rpy="1.57075 0 0" xyz="0 0 0"/>
+				<mass value="0.85"/>
+				<inertia
+					ixx="0.001" ixy="0" ixz="0"
+					iyy="0.001" iyz="0"
+					izz="0.001"/>
 			</inertial>
 		</link>
+		<gazebo reference="${prefix}_link">
+			<material>Gazebo/Grey</material>
+	    <mu1>1.0</mu1>
+	    <mu2>1.0</mu2>
+	    <kp>1000000.0</kp>
+	    <kd>100.0</kd>
+	    <minDepth>0.001</minDepth>
+	    <maxVel>1.0</maxVel>
+		</gazebo>
 		<joint name="${prefix}_joint" type="continuous">
 			<axis xyz="0 1 0"/>
@@ -28,6 +39,36 @@
 			<child link="${prefix}_link"/>
 			<origin rpy="${joint_roll} ${joint_pitch} ${joint_yaw}" xyz="${joint_x} ${joint_y} ${joint_z}"/>
-			<limit effort="100" velocity="100"/>
-			<joint_properties damping="0.0" friction="0.0"/>
+		</joint>
+		<link name="${prefix}tire_link">
+			<collision>
+				<origin rpy="1.57075 0 0" xyz="0 0 0"/>
+				<geometry>
+					<cylinder length="0.001" radius="0.001"/>
+				</geometry>
+			</collision>
+			<visual>
+				<origin rpy="0 0 ${pi/2}" xyz="0 0 0"/>
+				<geometry>
+					<mesh filename="package://evarobot_description/meshes/tire.stl" scale="1 1 1"/>
+				</geometry>
+				<material name="Black"/>
+			</visual>
+			<inertial>
+				<origin xyz="0 0 0" rpy="0 0 0"/>
+				<mass value="0.001"/>
+				<inertia
+					ixx="0.001" ixy="0" ixz="0"
+					iyy="0.001" iyz="0"
+					izz="0.001"/>
+			</inertial>
+		</link>
+		<gazebo reference="${prefix}tire_link">
+			<material>Gazebo/Black</material>
+		</gazebo>
+		<joint name="${prefix}tire_joint" type="continuous">
+			<axis xyz="0 1 0"/>
+			<parent link="${prefix}_link"/>
+			<child link="${prefix}tire_link"/>
+			<origin rpy="0 0 0" xyz="0.0 0.0 0.0"/>
 		</joint>
 	</xacro:macro>
