Commit message: modify for jade-devel

File: evarobot_description/urdf/evarobot.urdf.xacro (robot description, xacro)
@@ -1,11 +1,11 @@
-<?xml version="1.0"?>
+<?xml version="1.0" encoding="UTF-8" standalone="no" ?>
 <!--
   The complete evarobot library of xacros for easy reference
  -->
-<robot name="evarobot" xmlns:xacro="http://ros.org/wiki/xacro">
-  <xacro:property name="pi" value="3.1415926535897931" />
+<robot name="evarobot" xmlns:xacro="http://www.ros.org/wiki/xacro">
   <!-- Includes -->
   <xacro:include filename="$(find evarobot_description)/urdf/materials.urdf.xacro"/>
   <xacro:include filename="$(find evarobot_description)/urdf/evarobot_base.urdf.xacro"/>
+  <xacro:include filename="$(find evarobot_description)/urdf/evarobot_base_c.urdf.xacro"/>
   <xacro:include filename="$(find evarobot_description)/urdf/evarobot_caster.urdf.xacro"/>
   <xacro:include filename="$(find evarobot_description)/urdf/evarobot_wheel.urdf.xacro"/>
@@ -50,4 +50,14 @@
 					   box_y="0.30"
 					   box_z="0.30" />
+	<xacro:evarobot_base_c prefix="base"
+					   mesh_x="0.065"
+					   mesh_y="-0.11"
+					   mesh_z="-0.15"
+					   mesh_roll="0.0"
+					   mesh_pitch="0.0"
+					   mesh_yaw="0"
+					   box_x="0.40"
+					   box_y="0.30"
+					   box_z="0.30" />
   <!-- Left Wheel -->
   <xacro:evarobot_wheel prefix="left_wheel"
@@ -61,4 +71,7 @@
 						cylinder_radius="0.085"
 						parent_link="base_link" />
+<gazebo reference="orange_link">
+			<material>Gazebo/Orange</material>
+		</gazebo>
   <!-- Right Wheel 	 -->
   <xacro:evarobot_wheel prefix="right_wheel"

File: evarobot_description/urdf/evarobot_ahrs.urdf.xacro (robot description, xacro)
@@ -1,4 +1,4 @@
 <?xml version="1.0"?>
-<robot xmlns:xacro="http://ros.org/wiki/xacro">
+<robot xmlns:xacro="http://www.ros.org/wiki/xacro">
 	<xacro:macro name="evarobot_ahrs" params="prefix joint_x joint_y joint_z joint_roll joint_pitch joint_yaw parent_link topic_name frame_name update_rate service_name robot_namespace">
 		<link name="${prefix}_link">

File: evarobot_description/urdf/evarobot_base.urdf.xacro (robot description, xacro)
@@ -28,36 +28,4 @@
       <material>Gazebo/Black</material>
 		</gazebo>
-		<link name="${prefix}color_link">
-			<collision>
-				<origin xyz="0 0 0" rpy="0 0 0"/>
-				<geometry>
-					<box size="0.0001 0.0001 0.0001"/>
-				</geometry>
-			</collision>
-			<visual>
-				<origin xyz="${mesh_x} ${mesh_y} ${mesh_z}" rpy="${mesh_roll} ${mesh_pitch} ${mesh_yaw}" />
-				<geometry>
-					<mesh filename="package://evarobot_description/meshes/base_orange.stl" scale="1 1 1"/>
-				</geometry>
-				<material name="Orange" />
-			</visual>
-			<inertial>
-				<origin xyz="0 0 0" rpy="0 0 0"/>
-				<mass value="0.0001"/>
-				<inertia
-					ixx="1e-6" ixy="0.0" ixz="0.0"
-					iyy="1e-6" iyz="0.0"
-					izz="1e-6"/>
-			</inertial>
-		</link>
-		<gazebo reference="${prefix}color_link">
-      <material>Gazebo/Orange</material>
-		</gazebo>
-		<joint name="${prefix}color_joint" type="fixed">
-			<axis xyz="0 1 0" />
-			<origin xyz="0 0 0" rpy="0 0 0"/>
-			<parent link="${prefix}_link"/>
-			<child link="${prefix}color_link"/>
-		</joint>
 	</xacro:macro>
 </robot>

File: evarobot_description/urdf/evarobot_bumper.urdf.xacro (robot description, xacro)
@@ -1,4 +1,4 @@
-<?xml version="1.0"?>
-<robot xmlns:xacro="http://ros.org/wiki/xacro">
+<?xml version="1.0" encoding="UTF-8" standalone="no" ?>
+<robot xmlns:xacro="http://www.ros.org/wiki/xacro">
 	<xacro:macro name="evarobot_bumper"
 	params="prefix
@@ -8,6 +8,5 @@
 			topic_name
 			frame_name
-			*plate_name
-			">
+			*plate_name">
 		<!-- Bumper Link -->
 		<link name="${prefix}_link">

File: evarobot_description/urdf/evarobot_caster.urdf.xacro (robot description, xacro)
@@ -1,4 +1,4 @@
 <?xml version="1.0"?>
-<robot xmlns:xacro="http://ros.org/wiki/xacro">
+<robot xmlns:xacro="http://www.ros.org/wiki/xacro">
 	<xacro:macro name="evarobot_caster" params="prefix radius x y z roll pitch yaw axis_x axis_y axis_z parent_link">
     <link name="${prefix}_base_link">

File: evarobot_description/urdf/evarobot_infrared.urdf.xacro (robot description, xacro)
@@ -1,4 +1,4 @@
-<?xml version="1.0"?>
-<robot xmlns:xacro="http://ros.org/wiki/xacro">
+<?xml version="1.0" encoding="UTF-8" standalone="no" ?>
+<robot xmlns:xacro="http://www.ros.org/wiki/xacro">
 	<xacro:macro name="evarobot_infrared"
 		params="prefix
@@ -8,6 +8,5 @@
 				topic_name frame_name
 				update_rate
-				*plate_name
-				">
+				*plate_name">
 		<joint name="${prefix}_joint" type="fixed">
 				<axis xyz="1 0 0"/>

File: evarobot_description/urdf/evarobot_kinect.urdf.xacro (robot description, xacro)
@@ -1,4 +1,4 @@
-<?xml version="1.0"?>
-<robot xmlns:xacro="http://ros.org/wiki/xacro">
+<?xml version="1.0" encoding="UTF-8" standalone="no" ?>
+<robot xmlns:xacro="http://www.ros.org/wiki/xacro">
 	<xacro:macro name="evarobot_kinect"
 	params="prefix
@@ -6,6 +6,5 @@
 			parent_link
 			base_line update_rate
-			camera_name
-			">
+			camera_name">
     <joint name="camera_rgb_joint" type="fixed">
 			<origin xyz="0.0 -0.02 0.0" rpy="0.0 0.0 0.0"/>

File: evarobot_description/urdf/evarobot_lidar.urdf.xacro (robot description, xacro)
@@ -1,4 +1,4 @@
-<?xml version="1.0"?>
-<robot xmlns:xacro="http://ros.org/wiki/xacro">
+<?xml version="1.0" encoding="UTF-8" standalone="no" ?>
+<robot xmlns:xacro="http://www.ros.org/wiki/xacro">
 	<xacro:macro name="evarobot_lidar"
 	params="prefix joint_x joint_y joint_z joint_roll joint_pitch joint_yaw

File: evarobot_description/urdf/evarobot_sonar.urdf.xacro (robot description, xacro)
@@ -1,4 +1,4 @@
-<?xml version="1.0"?>
-<robot xmlns:xacro="http://ros.org/wiki/xacro">
+<?xml version="1.0" encoding="UTF-8" standalone="no" ?>
+<robot xmlns:xacro="http://www.ros.org/wiki/xacro">
 	<xacro:macro name="evarobot_sonar"
 	params="prefix
@@ -8,6 +8,5 @@
 			topic_name frame_name
 			update_rate
-			*plate_name
-			">
+			*plate_name">
 		<link name="${prefix}_link">
 			<inertial>

File: evarobot_description/urdf/evarobot_wheel.urdf.xacro (robot description, xacro)
@@ -1,4 +1,4 @@
 <?xml version="1.0"?>
-<robot name="evarobot" xmlns:xacro="http://ros.org/wiki/xacro">
+<robot name="evarobot" xmlns:xacro="http://www.ros.org/wiki/xacro">
 	<xacro:macro name="evarobot_wheel" params="prefix joint_x joint_y joint_z joint_roll joint_pitch joint_yaw cylinder_length cylinder_radius parent_link">
 		<link name="${prefix}_link">

File: evarobot_description/urdf/materials.urdf.xacro (robot description, xacro)
@@ -1,4 +1,4 @@
 <?xml version="1.0"?>
-<robot xmlns:xacro="http://ros.org/wiki/xacro">
+<robot xmlns:xacro="http://www.ros.org/wiki/xacro">
 	<!-- Materials -->
   <material name="Black">

File: evarobot_description/urdf/plates.urdf.xacro (robot description, xacro)
@@ -1,4 +1,4 @@
 <?xml version="1.0"?>
-<robot xmlns:xacro="http://ros.org/wiki/xacro">
+<robot xmlns:xacro="http://www.ros.org/wiki/xacro">
 <!-- Plates -->
 <xacro:property name="plate_0_0">
